Commit message: Fix robot spawning: remove duplicate pi definition, add nav2_minimal_tb4_description mesh path

File: cofetch_description/urdf/cofetch_robot.urdf.xacro (robot description, xacro)
@@ -1,29 +1,150 @@
 <?xml version="1.0"?>
 <robot name="cofetch_robot" xmlns:xacro="http://ros.org/wiki/xacro">
-  <xacro:include filename="$(find turtlebot4_description)/urdf/standard/turtlebot4.urdf.xacro" />
-  <xacro:property name="arm_x_offset" value="0.15"/>
-  <xacro:property name="arm_y_offset" value="0"/>
-  <xacro:property name="arm_z_offset" value="0.30"/>
-  <xacro:property name="arm_base_height" value="0.05"/>
-  <xacro:property name="arm_base_radius" value="0.04"/>
-  <xacro:property name="arm_base_mass" value="0.5"/>
+  <link name="base_footprint">
+    <visual>
+      <origin xyz="0 0 0" rpy="0 0 0"/>
+      <geometry>
+        <box size="0.001 0.001 0.001"/>
+      </geometry>
+    </visual>
+  </link>
+  <joint name="base_footprint_joint" type="fixed">
+    <parent link="base_footprint"/>
+    <child link="base_link"/>
+    <origin xyz="0 0 0.033" rpy="0 0 0"/>
+  </joint>
+  <link name="base_link">
+    <visual>
+      <origin xyz="0 0 0.0415" rpy="0 0 0"/>
+      <geometry>
+        <cylinder radius="0.17" length="0.083"/>
+      </geometry>
+      <material name="darkgrey">
+        <color rgba="0.2 0.2 0.2 1"/>
+      </material>
+    </visual>
+    <collision>
+      <origin xyz="0 0 0.0415" rpy="0 0 0"/>
+      <geometry>
+        <cylinder radius="0.17" length="0.083"/>
+      </geometry>
+    </collision>
+    <inertial>
+      <mass value="3.5"/>
+      <origin xyz="0 0 0.0415" rpy="0 0 0"/>
+      <inertia ixx="0.01" ixy="0" ixz="0" iyy="0.01" iyz="0" izz="0.01"/>
+    </inertial>
+  </link>
+  <gazebo reference="base_link">
+    <material>Gazebo/DarkGrey</material>
+  </gazebo>
+  <link name="top_plate_link">
+    <visual>
+      <origin xyz="0 0 0.003" rpy="0 0 0"/>
+      <geometry>
+        <cylinder radius="0.17" length="0.006"/>
+      </geometry>
+      <material name="white">
+        <color rgba="1 1 1 1"/>
+      </material>
+    </visual>
+    <collision>
+      <origin xyz="0 0 0.003" rpy="0 0 0"/>
+      <geometry>
+        <cylinder radius="0.17" length="0.006"/>
+      </geometry>
+    </collision>
+    <inertial>
+      <mass value="0.5"/>
+      <origin xyz="0 0 0.003" rpy="0 0 0"/>
+      <inertia ixx="0.001" ixy="0" ixz="0" iyy="0.001" iyz="0" izz="0.001"/>
+    </inertial>
+  </link>
+  <gazebo reference="top_plate_link">
+    <material>Gazebo/White</material>
+  </gazebo>
+  <joint name="top_plate_joint" type="fixed">
+    <parent link="base_link"/>
+    <child link="top_plate_link"/>
+    <origin xyz="0 0 0.086" rpy="0 0 0"/>
+  </joint>
+  <link name="rplidar_link">
+    <visual>
+      <origin xyz="0 0 0" rpy="0 0 0"/>
+      <geometry>
+        <cylinder radius="0.04" length="0.05"/>
+      </geometry>
+      <material name="black">
+        <color rgba="0.1 0.1 0.1 1"/>
+      </material>
+    </visual>
+    <collision>
+      <origin xyz="0 0 0" rpy="0 0 0"/>
+      <geometry>
+        <cylinder radius="0.04" length="0.05"/>
+      </geometry>
+    </collision>
+    <inertial>
+      <mass value="0.1"/>
+      <origin xyz="0 0 0" rpy="0 0 0"/>
+      <inertia ixx="0.0001" ixy="0" ixz="0" iyy="0.0001" iyz="0" izz="0.0001"/>
+    </inertial>
+  </link>
+  <gazebo reference="rplidar_link">
+    <material>Gazebo/Black</material>
+  </gazebo>
+  <joint name="rplidar_joint" type="fixed">
+    <parent link="top_plate_link"/>
+    <child link="rplidar_link"/>
+    <origin xyz="0 0 0.035" rpy="0 0 0"/>
+  </joint>
+  <link name="camera_link">
+    <visual>
+      <origin xyz="0 0 0" rpy="0 0 0"/>
+      <geometry>
+        <box size="0.03 0.08 0.03"/>
+      </geometry>
+      <material name="black">
+        <color rgba="0.1 0.1 0.1 1"/>
+      </material>
+    </visual>
+    <collision>
+      <origin xyz="0 0 0" rpy="0 0 0"/>
+      <geometry>
+        <box size="0.03 0.08 0.03"/>
+      </geometry>
+    </collision>
+    <inertial>
+      <mass value="0.05"/>
+      <origin xyz="0 0 0" rpy="0 0 0"/>
+      <inertia ixx="0.00001" ixy="0" ixz="0" iyy="0.00001" iyz="0" izz="0.00001"/>
+    </inertial>
+  </link>
+  <gazebo reference="camera_link">
+    <material>Gazebo/Black</material>
+  </gazebo>
+  <joint name="camera_joint" type="fixed">
+    <parent link="top_plate_link"/>
+    <child link="camera_link"/>
+    <origin xyz="0 0.06 0.015" rpy="0 0 0"/>
+  </joint>
   <link name="arm_base_link">
     <visual>
       <origin xyz="0 0 0" rpy="0 0 0"/>
       <geometry>
-        <cylinder radius="${arm_base_radius}" length="${arm_base_height}"/>
+        <cylinder radius="0.04" length="0.05"/>
       </geometry>
       <material name="grey">
-        <color rgba="0.5 0.5 0.5 1.0"/>
-      </material>
-    </visual>
-    <collision>
-      <origin xyz="0 0 0" rpy="0 0 0"/>
-      <geometry>
-        <cylinder radius="${arm_base_radius}" length="${arm_base_height}"/>
-      </geometry>
-    </collision>
-    <inertial>
-      <mass value="${arm_base_mass}"/>
+        <color rgba="0.5 0.5 0.5 1"/>
+      </material>
+    </visual>
+    <collision>
+      <origin xyz="0 0 0" rpy="0 0 0"/>
+      <geometry>
+        <cylinder radius="0.04" length="0.05"/>
+      </geometry>
+    </collision>
+    <inertial>
+      <mass value="0.5"/>
       <origin xyz="0 0 0" rpy="0 0 0"/>
       <inertia ixx="0.001" ixy="0" ixz="0" iyy="0.001" iyz="0" izz="0.001"/>
@@ -34,7 +155,7 @@
   </gazebo>
   <joint name="arm_base_joint" type="fixed">
-    <parent link="shell_link"/>
+    <parent link="top_plate_link"/>
     <child link="arm_base_link"/>
-    <origin xyz="${arm_x_offset} ${arm_y_offset} ${arm_z_offset}" rpy="0 0 0"/>
+    <origin xyz="0.15 0 0.03" rpy="0 0 0"/>
   </joint>
   <link name="arm_link_1">
@@ -45,5 +166,5 @@
       </geometry>
       <material name="orange">
-        <color rgba="1.0 0.5 0.0 1.0"/>
+        <color rgba="1.0 0.5 0.0 1"/>
       </material>
     </visual>
@@ -66,5 +187,5 @@
     <parent link="arm_base_link"/>
     <child link="arm_link_1"/>
-    <origin xyz="0 0 ${arm_base_height}" rpy="0 0 0"/>
+    <origin xyz="0 0 0.05" rpy="0 0 0"/>
     <axis xyz="0 0 1"/>
     <limit lower="-3.14159" upper="3.14159" effort="100" velocity="1.0"/>
@@ -77,5 +198,5 @@
       </geometry>
       <material name="orange">
-        <color rgba="1.0 0.5 0.0 1.0"/>
+        <color rgba="1.0 0.5 0.0 1"/>
       </material>
     </visual>
@@ -109,5 +230,5 @@
       </geometry>
       <material name="darkgrey">
-        <color rgba="0.3 0.3 0.3 1.0"/>
+        <color rgba="0.3 0.3 0.3 1"/>
       </material>
     </visual>
@@ -139,5 +260,5 @@
       </geometry>
       <material name="black">
-        <color rgba="0.1 0.1 0.1 1.0"/>
+        <color rgba="0.1 0.1 0.1 1"/>
       </material>
     </visual>
@@ -171,5 +292,5 @@
       </geometry>
       <material name="black">
-        <color rgba="0.1 0.1 0.1 1.0"/>
+        <color rgba="0.1 0.1 0.1 1"/>
       </material>
     </visual>
@@ -203,5 +324,5 @@
       </geometry>
       <material name="blue">
-        <color rgba="0.0 0.0 1.0 1.0"/>
+        <color rgba="0.0 0.0 1.0 1"/>
       </material>
     </visual>

Commit message: Use standalone URDF without external mesh dependencies
- cofetch_robot.urdf.xacro: standalone model using basic geometries (cylinder, box, sphere)
- gazebo.launch.py: simplified model_paths (only irobot_create meshes)

File: cofetch_description/urdf/cofetch_robot.urdf.xacro (robot description, xacro)
@@ -127,5 +127,5 @@
     <parent link="top_plate_link"/>
     <child link="camera_link"/>
-    <origin xyz="0 0.06 0.015" rpy="0 0 0"/>
+    <origin xyz="0.06 0 0.015" rpy="0 0 0"/>
   </joint>
   <link name="arm_base_link">
